Commit message: Update mycontroller.urdf

File: urdf/mycontroller.urdf (robot description, URDF)
Before this commit: robot firefighter, 15 links, 14 joints
Links:
- link base: geometry collision mesh filename=package://base.dae; visual mesh filename=package://base.dae
- link link1: geometry collision mesh filename=package://link1.dae; visual mesh filename=package://link1.dae
- link link10: geometry collision mesh filename=package://link3.dae; visual mesh filename=package://link3.dae
- link link11: geometry collision mesh filename=package://link4.dae; visual mesh filename=package://link4.dae
- link link12: geometry collision mesh filename=package://link5.dae; visual mesh filename=package://link5.dae
- link link13: geometry collision mesh filename=package://link6.dae; visual mesh filename=package://link6.dae
- link link14: geometry collision mesh filename=package://link7.dae; visual mesh filename=package://link7.dae
- link link2: geometry collision mesh filename=package://link2.dae; visual mesh filename=package://link2.dae
- link link3: geometry collision mesh filename=package://link3.dae; visual mesh filename=package://link3.dae
- link link4: geometry collision mesh filename=package://link4.dae; visual mesh filename=package://link4.dae
- link link5: geometry collision mesh filename=package://link5.dae; visual mesh filename=package://link5.dae
- link link6: geometry collision mesh filename=package://link6.dae; visual mesh filename=package://link6.dae
- link link7: geometry collision mesh filename=package://link7.dae; visual mesh filename=package://link7.dae
- link link8: geometry collision mesh filename=package://link1.dae; visual mesh filename=package://link1.dae
- link link9: geometry collision mesh filename=package://link2.dae; visual mesh filename=package://link2.dae
